File: power-iot-meter-pcb/power-iot-meter-pcb.kicad_pcb (KiCad board)
At the start: 2 copper layers, 119.8 x 64.2 mm, 9 parts, among them J1 AC OUTPUT, J2 AC Current Sensor, J3 AC INPUT, J4 AC Voltage Sensor, J5 POWER_FEMALE, J6 POWER_MALE, J7 UART_FEMALE, U1 ESP32-DEVKIT-V1

Commit message: PCB update
Parts:
- added C1: 100uF, Capacitor_THT:CP_Radial_D8.0mm_P3.50mm, F.Cu at (120.0, 104.8)
- added J8: VOLTAGE_CURRENT, Connector_PinSocket_2.00mm:PinSocket_1x06_P2.00mm_Vertical, F.Cu at (115.0, 114.6)
- added R1: 10k, Resistor_THT:R_Axial_DIN0207_L6.3mm_D2.5mm_P10.16mm_Horizontal, F.Cu at (102.0, 116.6)
- added R2: 10k, Resistor_THT:R_Axial_DIN0207_L6.3mm_D2.5mm_P10.16mm_Horizontal, F.Cu at (102.0, 109.8)
- added R3: 10k, Resistor_THT:R_Axial_DIN0207_L6.3mm_D2.5mm_P10.16mm_Horizontal, F.Cu at (112.2, 113.4)
- added R4: 10k, Resistor_THT:R_Axial_DIN0207_L6.3mm_D2.5mm_P10.16mm_Horizontal, F.Cu at (112.2, 120.6)
- added R5: 10k, Resistor_THT:R_Axial_DIN0207_L6.3mm_D2.5mm_P10.16mm_Horizontal, F.Cu at (102.0, 127.0)
- added R6: 10k, Resistor_THT:R_Axial_DIN0207_L6.3mm_D2.5mm_P10.16mm_Horizontal, F.Cu at (112.2, 123.8)
- renumbered J5 to J1, J1 to J2, J2 to J3, J3 to J4, J6 to J5, J4 to J6
Connections:
- net AC_IN1 renamed Net-(J2-Pad2)
- net AC_IN2 renamed Net-(J3-Pad2)
- net AC_OUT1 renamed Net-(J2-Pad1)
- net Rx renamed PZEM_TX_PIN
- net Tx renamed PZEM_RX_PIN
- U1 pad 17: Net-(U1-Pad17) -> VOLTAGE
- U1 pad 18: Net-(U1-Pad18) -> CURRENT
Routing:
- net VOLTAGE: track 0.00 -> 81.3 mm
- net CURRENT: track 0.00 -> 80.4 mm
- net GND: track 109.7 -> 181.5 mm
- net +5V: track 88.8 -> 127.1 mm
- net Net-(J8-Pad5): track 0.00 -> 6.18 mm
- net Net-(J8-Pad2): track 0.00 -> 6.00 mm
