File: power-iot-meter-pcb/power-iot-meter-pcb.sch (KiCad schematic (older format))
At the start: 9 parts, among them J1 AC OUTPUT, J2 AC Current Sensor, J3 AC INPUT, J4 AC Voltage Sensor, J5 POWER_FEMALE, J6 POWER_MALE, J7 UART_FEMALE, U1 ESP32-DEVKIT-V1

Commit message: PCB update
Parts:
- added C1: 100uF, Capacitor_THT:CP_Radial_D8.0mm_P3.50mm, symbol Device:CP
- added J8: VOLTAGE_CURRENT, Connector_PinSocket_2.00mm:PinSocket_1x06_P2.00mm_Vertical, symbol Connector:Conn_01x06_Female
- added R1, R2, R3, R4, R5, R6: 10k, Resistor_THT:R_Axial_DIN0207_L6.3mm_D2.5mm_P10.16mm_Horizontal, symbol Device:R
- renumbered J5 to J1, J1 to J2, J2 to J3, J3 to J4, J6 to J5, J4 to J6
Connections:
- net +5V: now also C1.1, J8.1 (Pin_1), J8.6 (Pin_6)
- net GND: now also C1.2, J8.3 (Pin_3), J8.4 (Pin_4), R2.2, R5.2
- net VOLTAGE: now reaches U1.17 (VP)
- net VOLTAGE: now also R1.1, R2.1, R3.2
- net CURRENT: now reaches U1.18 (VN)
- net CURRENT: now also R4.2, R5.1, R6.2
- net AC_IN1: no longer names the net of J2.2 (Pin_2), J4.1 (Pin_1), J6.1 (Pin_1), PS1.1 (AC1)
- net AC_IN2: no longer names the net of J3.2 (Pin_2), J4.2 (Pin_2), J6.2 (Pin_2), PS1.2 (AC2)
- net AC_OUT1: no longer names the net of J2.1 (Pin_1), J3.1 (Pin_1)
- net Rx renamed PZEM_TX_PIN
- net Tx renamed PZEM_RX_PIN
- new net: J8.2 (Pin_2), R1.2, R3.1
- new net: J8.5 (Pin_5), R4.1, R6.1
Other:
- moved on the sheet: J1, J2, J3, J4, J5, J6, J7, PS1
